File: KiCad/436.5MHz LNA/436.5MHz LNA.kicad_pcb (KiCad board)
At the start: 2 copper layers, 33.3 x 13.5 mm, 15 parts, among them J1 Conn_Coaxial, J2 Conn_Coaxial, J3 +9V, Q1 J310

Commit message: no pushes from yesterday seem to have worked. Extended soldermask on rf path
Other:
- board text added: "436.5MHz LNA v1.1"
- board text removed: "436.5MHz LNA"
Changed lines of the file:
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@@
     (effects (font (size 0.5 0.5) (thickness 0.125)))
   )
-  (gr_text "436.5MHz LNA\n" (at 100.95 68.5) (layer "F.SilkS")
+  (gr_text "436.5MHz LNA v1.1\n" (at 100.95 68.5) (layer "F.SilkS")
     (effects (font (size 1 1) (thickness 0.15)))
   )
@@
   (zone (net 0) (net_name "") (layer "F.Mask") (hatch full 0.508)
     (connect_pads (clearance 0.508))
-    (min_thickness 0.254) (filled_areas_thickness no)
-    (fill yes (thermal_gap 0.508) (thermal_bridge_width 0.508))
-    (polygon
-      (pts
-        (xy 102.2 74)
-        (xy 101.75 74)
-        (xy 101.75 72)
-        (xy 102.2 72)
-      )
-    )
-  )
-  (zone (net 0) (net_name "") (layer "F.Mask") (hatch full 0.508)
-    (connect_pads (clearance 0.508))
-    (min_thickness 0.254) (filled_areas_thickness no)
-    (fill yes (thermal_gap 0.508) (thermal_bridge_width 0.508))
-    (polygon
-      (pts
-        (xy 106.8 74)
-        (xy 106.35 74)
-        (xy 106.35 72)
-        (xy 106.8 72)
+    (min_thickness 0.1016) (filled_areas_thickness no)
+    (fill yes (thermal_gap 0.508) (thermal_bridge_width 0.508))
+    (polygon
+      (pts
+        (xy 102.15 74)
+        (xy 101.8 74)
+        (xy 101.8 72)
+        (xy 102.15 72)
+      )
+    )
+  )
+  (zone (net 0) (net_name "") (layer "F.Mask") (hatch full 0.508)
+    (connect_pads (clearance 0.508))
+    (min_thickness 0.1016) (filled_areas_thickness no)
+    (fill yes (thermal_gap 0.508) (thermal_bridge_width 0.508))
+    (polygon
+      (pts
+        (xy 106.75 74)
+        (xy 106.4 74)
+        (xy 106.4 72)
+        (xy 106.75 72)
       )
     )
@@
   (zone (net 0) (net_name "") (layer "F.Mask") (hatch full 0.508)
     (connect_pads (clearance 0.508))
-    (min_thickness 0.254) (filled_areas_thickness no)
-    (fill yes (thermal_gap 0.508) (thermal_bridge_width 0.508))
-    (polygon
-      (pts
-        (xy 94.15 74)
-        (xy 93.7 74)
-        (xy 93.7 72)
-        (xy 94.15 72)
-      )
-    )
-  )
-  (zone (net 0) (net_name "") (layer "F.Mask") (hatch full 0.508)
-    (connect_pads (clearance 0.508))
-    (min_thickness 0.254) (filled_areas_thickness no)
-    (fill yes (thermal_gap 0.508) (thermal_bridge_width 0.508))
-    (polygon
-      (pts
-        (xy 108.35 74)
-        (xy 107.9 74)
-        (xy 107.9 72)
-        (xy 108.35 72)
+    (min_thickness 0.1016) (filled_areas_thickness no)
+    (fill yes (thermal_gap 0.508) (thermal_bridge_width 0.508))
+    (polygon
+      (pts
+        (xy 94.1 74)
+        (xy 93.75 74)
+        (xy 93.75 72)
+        (xy 94.1 72)
+      )
+    )
+  )
+  (zone (net 0) (net_name "") (layer "F.Mask") (hatch full 0.508)
+    (connect_pads (clearance 0.508))
+    (min_thickness 0.1016) (filled_areas_thickness no)
+    (fill yes (thermal_gap 0.508) (thermal_bridge_width 0.508))
+    (polygon
+      (pts
+        (xy 108.3 74)
+        (xy 107.95 74)
+        (xy 107.95 72)
+        (xy 108.3 72)
       )
     )
@@
   (zone (net 0) (net_name "") (layer "F.Mask") (hatch full 0.508)
     (connect_pads (clearance 0.508))
-    (min_thickness 0.254) (filled_areas_thickness no)
+    (min_thickness 0.1016) (filled_areas_thickness no)
     (fill yes (thermal_gap 0.508) (thermal_bridge_width 0.508))
     (polygon
       (pts
         (xy 112.3 74)
-        (xy 110.95 74)
-        (xy 110.95 72)
+        (xy 111 74)
+        (xy 111 72)
         (xy 112.3 72)
       )
@@
   (zone (net 0) (net_name "") (layer "F.Mask") (hatch full 0.508)
     (connect_pads (clearance 0.508))
-    (min_thickness 0.254) (filled_areas_thickness no)
-    (fill yes (thermal_gap 0.508) (thermal_bridge_width 0.508))
-    (polygon
-      (pts
-        (xy 99.15 74)
-        (xy 98.55 74)
-        (xy 98.55 72)
-        (xy 99.15 72)
-      )
-    )
-  )
-  (zone (net 0) (net_name "") (layer "F.Mask") (hatch full 0.508)
-    (connect_pads (clearance 0.508))
-    (min_thickness 0.254) (filled_areas_thickness no)
-    (fill yes (thermal_gap 0.508) (thermal_bridge_width 0.508))
-    (polygon
-      (pts
-        (xy 95.85 74)
-        (xy 95.25 74)
-        (xy 95.25 72)
-        (xy 95.85 72)
+    (min_thickness 0.1016) (filled_areas_thickness no)
+    (fill yes (thermal_gap 0.508) (thermal_bridge_width 0.508))
+    (polygon
+      (pts
+        (xy 99.1 74)
+        (xy 98.6 74)
+        (xy 98.6 72)
+        (xy 99.1 72)
+      )
+    )
+  )
+  (zone (net 0) (net_name "") (layer "F.Mask") (hatch full 0.508)
+    (connect_pads (clearance 0.508))
+    (min_thickness 0.1016) (filled_areas_thickness no)
+    (fill yes (thermal_gap 0.508) (thermal_bridge_width 0.508))
+    (polygon
+      (pts
+        (xy 95.8 74)
+        (xy 95.3 74)
+        (xy 95.3 72)
+        (xy 95.8 72)
       )
     )
@@
   (zone (net 0) (net_name "") (layer "F.Mask") (hatch full 0.508)
     (connect_pads (clearance 0.508))
-    (min_thickness 0.254) (filled_areas_thickness no)
-    (fill yes (thermal_gap 0.508) (thermal_bridge_width 0.508))
-    (polygon
-      (pts
-        (xy 103.75 74)
-        (xy 103.3 74)
-        (xy 103.3 72)
-        (xy 103.75 72)
+    (min_thickness 0.1016) (filled_areas_thickness no)
+    (fill yes (thermal_gap 0.508) (thermal_bridge_width 0.508))
+    (polygon
+      (pts
+        (xy 103.7 74)
+        (xy 103.35 74)
+        (xy 103.35 72)
+        (xy 103.7 72)
       )
     )
@@
   (zone (net 0) (net_name "") (layer "F.Mask") (hatch full 0.508)
     (connect_pads (clearance 0.508))
-    (min_thickness 0.254) (filled_areas_thickness no)
-    (fill yes (thermal_gap 0.508) (thermal_bridge_width 0.508))
-    (polygon
-      (pts
-        (xy 91.1 74)
+    (min_thickness 0.1016) (filled_areas_thickness no)
+    (fill yes (thermal_gap 0.508) (thermal_bridge_width 0.508))
+    (polygon
+      (pts
+        (xy 91.05 74)
         (xy 89.75 74)
         (xy 89.75 72)
-        (xy 91.1 72)
-      )
-    )
+        (xy 91.05 72)
+      )
+    )

Commit message: flipped the JFET so the gate has a more common ground with the RF path
Parts:
- C4: value 2.8p -> 1.2p
- J1, J2: value Conn_Coaxial -> Coaxial SMA
- L1: value 22n -> 36n
- L2, L3: value 25n -> 39n
- R1: value 200 -> 100
- R2: value 200 -> 5.1
- moved Q1 1.90 mm to (97.2, 74.0), turned to -90 degrees
Connections:
- Q1 pad 1: Net-(C1-Pad2) -> Net-(Q1-Pad1)
- Q1 pad 2: Net-(Q1-Pad2) -> Net-(C1-Pad2)
- R2 pad 1: Net-(Q1-Pad2) -> Net-(Q1-Pad1)
Routing:
- net Net-(Q1-Pad2): track 1.48 -> 0.00 mm
- net Net-(Q1-Pad1): track 0.00 -> 1.48 mm
